File: Hardware/Placa PCB e Esquema/Placa PCB e Esquema.kicad_sch (KiCad schematic)
At the start: 39 parts, among them J1 PT1000, J2 Alimentação, J3 Celula de Peltier, J4 Ventoinhas, K1 FINDER-40.52, Q1 Q_NMOS_GDS, Q2 Q_NMOS_GDS, U1 TL084, U2 TL084, U3 XIAO_ESP32C3

Commit message: Prototipo Funcional V4
Connections:
- net Aquecer/Arrefecer: now also Q2.1 (G), R19.1, U3.3 (D2); no longer Q1.1 (G), R20.2, U3.2 (D1)
- net Controle Celula: now also Q1.1 (G), R20.2, U3.2 (D1); no longer Q2.1 (G), R19.1, U3.3 (D2)
Changed lines of the file:
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@@
 		)
 	)
-	(label "Controle Celula"
+	(label "Aquecer{slash}Arrefecer"
 		(at 20.32 158.75 0)
 		(effects
@@
 		)
 	)
-	(label "Aquecer{slash}Arrefecer"
+	(label "Controle Celula"
 		(at 214.63 87.63 0)
 		(effects
@@
 		)
 	)
-	(label "Aquecer{slash}Arrefecer"
+	(label "Controle Celula"
 		(at 24.13 185.42 0)
 		(effects
@@
 		)
 	)
-	(label "Controle Celula"
+	(label "Aquecer{slash}Arrefecer"
 		(at 215.9 132.08 0)
 		(effects
